File: hardware/design-files/ct_sensor.kicad_sch (KiCad schematic)
At the start: 10 parts, among them J2 SCT-013-030, U5 ADS1115IDGS

Commit message: feat(hardware): update KiCad schematics with component symbols and layout refinements
- Add ADS1115 16-bit I2C ADC symbol to CT sensor schematic
- Add AudioJack2 connector symbol for analog signal input
- Update ESP32 module schematic with refined pin configurations
- Update power supply schematic with improved component placement
- Update relay driver schematic with optimized routing
- Refine PCB layout in gateway.kicad_pcb with better trace routing
- Update project settings in gateway.kicad_pro for design rule compliance
- Add project rules configuration in gateway.kicad_prl for manufacturing constraints
Parts:
- removed C5: 10uF, Capacitor_SMD:C_0805_2012Metric, symbol Device:C
- removed D2, D3: BAT54, Diode_SMD:D_SOD-323, symbol Device:D_Schottky
- removed J2: SCT-013-030, Connector_Audio:Jack_3.5mm_Horizontal, symbol Connector:AudioJack2
- removed R1: 33R 1%, Resistor_SMD:R_0805_2012Metric, symbol Device:R
- removed R4: 1K, Resistor_SMD:R_0805_2012Metric, symbol Device:R
- added J2: SCT-013-030, Connector_PinHeader_2.54mm:PinHeader_1x02_P2.54mm_Vertical, symbol Connector_Audio:AudioJack2
Connections:
- net GND: now also C4.2, R3.2, U5.1 (ADDR), U5.3 (GND)
- net I2C_SCL: now also U5.10 (SCL)
- net I2C_SDA: now also U5.9 (SDA)
- new net: C4.1, J2.T, R2.2, R3.1
- new net: J2.S, U5.4 (AIN0)
- new net +3.3V: R2.1, U5.8 (VDD)
- no-connect marks 0 -> 4

Commit message: feat(hardware): update PCB layout and component footprints
- Reposition ADS1115 ADC module on PCB (moved from 84.35,28 to 60.5,49.35 with 180° rotation)
- Update CT sensor connector footprint from PinHeader to 3.5mm audio jack (Switronic ST-005-G)
- Correct ESP32 module connector footprint from 1x02 to 1x06 pin header
- Regenerate component UUIDs and silk screen coordinates to reflect new placements
- Optimize PCB layout for improved signal routing and component accessibility
Parts:
- J2: footprint Connector_PinHeader_2.54mm:PinHeader_1x02_P2.54mm_Vertical -> Connector_Audio:Jack_3.5mm_Switronic_ST-005-G_horizontal
Changed lines of the file:
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@@
 			)
 		)
-		(property "Footprint" "Connector_PinHeader_2.54mm:PinHeader_1x02_P2.54mm_Vertical"
+		(property "Footprint" "Connector_Audio:Jack_3.5mm_Switronic_ST-005-G_horizontal"
 			(at 58.42 76.2 0)
 			(hide yes)
