File: hardware/design-files/esp32_module.kicad_sch (KiCad schematic)
At the start: 10 parts, among them J4 UART_HDR, SW1 BOOT, SW2 RESET, U4 ESP32-WROOM-32

Commit message: feat(hardware): update KiCad schematics with component symbols and layout refinements
- Add ADS1115 16-bit I2C ADC symbol to CT sensor schematic
- Add AudioJack2 connector symbol for analog signal input
- Update ESP32 module schematic with refined pin configurations
- Update power supply schematic with improved component placement
- Update relay driver schematic with optimized routing
- Refine PCB layout in gateway.kicad_pcb with better trace routing
- Update project settings in gateway.kicad_pro for design rule compliance
- Add project rules configuration in gateway.kicad_prl for manufacturing constraints
Parts:
- removed C6: 100nF, Capacitor_SMD:C_0402_1005Metric, symbol Device:C
- removed C7: 10uF, Capacitor_SMD:C_0805_2012Metric, symbol Device:C
- removed D7: LED_Blue, LED_SMD:LED_0805_2012Metric, symbol Device:LED
- removed D8: PESD3V3L1BA, Diode_SMD:D_SOD-323, symbol Device:D_TVS
- removed J4: UART_HDR, Connector_PinHeader_2.54mm:PinHeader_1x04_P2.54mm_Vertical, symbol Connector:Conn_01x04_Pin
- removed R8: 10K, Resistor_SMD:R_0805_2012Metric, symbol Device:R
- removed R9: 1K, Resistor_SMD:R_0805_2012Metric, symbol Device:R
- removed SW1: BOOT, Button_Switch_SMD:SW_SPST_TL3342, symbol Switch:SW_Push
- removed SW2: RESET, Button_Switch_SMD:SW_SPST_TL3342, symbol Switch:SW_Push
- removed U4: ESP32-WROOM-32, RF_Module:ESP32-WROOM-32, symbol RF_Module:ESP32-WROOM-32
- added U4: ESP32 DevKit, Connector_PinHeader_2.54mm:PinHeader_1x02_P2.54mm_Vertical, symbol Connector_Generic:Conn_01x06
Connections:
- net GND: now also U4.2 (Pin_2)
- net GPIO_RELAY: now also U4.5 (Pin_5)
- net I2C_SCL: now also U4.3 (Pin_3)
- net I2C_SDA: now also U4.4 (Pin_4)
- net VCC_3V3: now also U4.1 (Pin_1)
- no-connect marks 0 -> 1
Other:
- note added: "3V3"
- note added: "GND"
- note added: "GPIO 18 (Relay)"
- note added: "GPIO 21 (SDA)"
- note added: "GPIO 22 (SCL)"

Commit message: feat(hardware): update PCB layout and component footprints
- Reposition ADS1115 ADC module on PCB (moved from 84.35,28 to 60.5,49.35 with 180° rotation)
- Update CT sensor connector footprint from PinHeader to 3.5mm audio jack (Switronic ST-005-G)
- Correct ESP32 module connector footprint from 1x02 to 1x06 pin header
- Regenerate component UUIDs and silk screen coordinates to reflect new placements
- Optimize PCB layout for improved signal routing and component accessibility
Parts:
- U4: footprint Connector_PinHeader_2.54mm:PinHeader_1x02_P2.54mm_Vertical -> Connector_PinHeader_2.54mm:PinHeader_1x06_P2.54mm_Vertical
Changed lines of the file:
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@@
 			)
 		)
-		(property "Footprint" "Connector_PinHeader_2.54mm:PinHeader_1x02_P2.54mm_Vertical"
+		(property "Footprint" "Connector_PinHeader_2.54mm:PinHeader_1x06_P2.54mm_Vertical"
 			(at 95.25 62.23 0)
 			(hide yes)
